Commit message: fix (Robot.urdf.xacro) the distance with base_link with link1 1. change 0.275 to 0.375

File: TestRos/src/TestInput/urdf/xacro/Robot.urdf.xacro (robot description, xacro)
@@ -36,6 +36,6 @@
         <parent link="base_link"/>
         <child link="link_1"/>
-        <origin xyz="0 0 0.275" rpy="${-PI/2} 0 0"/>
-        <axis xyz="0 0 1"/>
+        <origin xyz="0 0 0.375" rpy="${-PI/2} 0 0"/>
+        <axis xyz="0 1 0"/>
     </joint>
     <link name="link_2">

Commit message: fix (Robot.urdf.xacro) the distance with base_link with link1 1.在launch文件中取消Joint_states 的发送方

File: TestRos/src/TestInput/urdf/xacro/Robot.urdf.xacro (robot description, xacro)
@@ -33,5 +33,5 @@
         </visual>
     </link>
-    <joint name="baseTolink1" type="continuous">
+    <joint name="BaseToLink_1" type="continuous">
         <parent link="base_link"/>
         <child link="link_1"/>
@@ -50,5 +50,5 @@
         </visual>
     </link>
-    <joint name="link1Tolink2" type="continuous">
+    <joint name="Link_1ToLink_2" type="continuous">
         <parent link="link_1"/>
         <child link="link_2"/>
@@ -67,5 +67,5 @@
         </visual>
     </link>
-    <joint name="link_2Tolink_3" type="continuous">
+    <joint name="Link_2ToLink_3" type="continuous">
         <parent link="link_2"/>
         <child link="link_3"/>
@@ -84,5 +84,5 @@
         </visual>
     </link>
-    <joint name="link_3Tolink_4" type="continuous">
+    <joint name="Link_3ToLink_4" type="continuous">
         <parent link="link_3"/>
         <child link="link_4"/>
@@ -101,5 +101,5 @@
         </visual>
     </link>
-    <joint name="link_4Tolink_5" type="continuous">
+    <joint name="Link_4ToLink_5" type="continuous">
         <parent link="link_4"/>
         <child link="link_5"/>
@@ -118,5 +118,5 @@
         </visual>
     </link>
-    <joint name="link_5Tolink_6" type="continuous">
+    <joint name="Link_5ToLink_6" type="continuous">
         <parent link="link_5"/>
         <child link="link_6"/>
