Commit message: feat (Testinput) add model

File: TestRos/src/TestInput/urdf/ShowModel.urdf (robot description, URDF)
Before this commit: robot mymodel, 1 links, 0 joints
Links:
- link base_link: geometry visual mesh filename=package://TestInput/urdf/model/1.STL

File: TestRos/src/TestInput/urdf/xacro/Robot.urdf.xacro (robot description, xacro)
@@ -2,10 +2,11 @@
 <robot name="mycar" xmlns:xacro="http://wiki.ros.org/xacro">
     <xacro:property name="PI" value="3.1415926"/>
-    <xacro:property name="TrolleyPath" value="package://TestInputModel/urdf/Trolley.stl"/>
-    <xacro:property name="Link1Path" value="package://TestInputModel/urdf/Link1.stl"/>
-    <xacro:property name="Link2Path" value="package://TestInputModel/urdf/Link2.stl"/>
-    <xacro:property name="Link3Path" value="package://TestInputModel/urdf/Link3.stl"/>
-    <xacro:property name="Link4Path" value="package://TestInputModel/urdf/Link4.stl"/>
-    <xacro:property name="Link5Path" value="package://TestInputModel/urdf/Link5.stl"/>
+    <xacro:property name="TrolleyPath" value="package://TestInput/urdf/model/1.STL"/>
+    <xacro:property name="Link1Path" value="package://TestInput/urdf/model/2.STL"/>
+    <xacro:property name="Link2Path" value="package://TestInput/urdf/model/3.STL"/>
+    <xacro:property name="Link3Path" value="package://TestInput/urdf/model/4.STL"/>
+    <xacro:property name="Link4Path" value="package://TestInput/urdf/model/5.STL"/>
+    <xacro:property name="Link5Path" value="package://TestInput/urdf/model/6.STL"/>
+    <xacro:property name="Link6Path" value="package://TestInput/urdf/model/7.STL"/>
     <link name="base_link">
         <visual>
@@ -35,5 +36,5 @@
         <parent link="base_link"/>
         <child link="link_1"/>
-        <origin xyz="0 0 0" rpy="0 0 0"/>
+        <origin xyz="0 0 0.275" rpy="${-PI/2} 0 0"/>
         <axis xyz="0 0 1"/>
     </joint>
@@ -52,5 +53,5 @@
         <parent link="link_1"/>
         <child link="link_2"/>
-        <origin xyz="0.0 0.0 0.0" rpy="-1.571 -1.571 0"/>
+        <origin xyz="0.0 0.0 0.0" rpy="0 0 0"/>
         <axis xyz="0 0 1"/>
     </joint>
@@ -69,5 +70,5 @@
         <parent link="link_2"/>
         <child link="link_3"/>
-        <origin xyz="0.4 0.0 0.02" rpy="0 0 1.571"/>
+        <origin xyz="0 -0.4 0.02" rpy="0 0 0"/>
         <axis xyz="0 0 1"/>
     </joint>
@@ -86,5 +87,5 @@
         <parent link="link_3"/>
         <child link="link_4"/>
-        <origin xyz="0 -0.45 0" rpy="1.571 0 0"/>
+        <origin xyz="0 0 0" rpy="${PI/2} 0 0"/>
         <axis xyz="0 0 1"/>
     </joint>
@@ -103,5 +104,22 @@
         <parent link="link_4"/>
         <child link="link_5"/>
-        <origin xyz="0 0 0" rpy="-1.571 0 0"/>
+        <origin xyz="0 0 0.45" rpy="${-PI/2} 0 0"/>
+        <axis xyz="0 0 1"/>
+    </joint>
+    <link name="link_6">
+        <visual>
+            <geometry>
+                <mesh filename="${Link6Path}"/>
+            </geometry>
+            <origin xyz="0 0 0" rpy="0 0 0"/>
+            <material name="red">
+                <color rgba="1 1 1 1"/>
+            </material>
+        </visual>
+    </link>
+    <joint name="link_5Tolink_6" type="continuous">
+        <parent link="link_5"/>
+        <child link="link_6"/>
+        <origin xyz="0 -0.07 0" rpy="${PI/2} 0 0"/>
         <axis xyz="0 0 1"/>
     </joint>

Commit message: feat(add other library)

File: TestRos/src/TestInput/urdf/ShowModel.urdf (robot description, URDF)
Before this commit: robot mymodel, 1 links, 0 joints
Links:
- added link link_1; visual mesh filename=package://TestInput/urdf/model/2.STL
