Commit message: feat(add other package)

File: TestRos/src/model_source/urdf/xacro/robot_model.urdf.xacro (robot description, xacro)
@@ -2,16 +2,15 @@
 <robot name="mycar" xmlns:xacro="http://wiki.ros.org/xacro">
     <xacro:property name="PI" value="3.1415926"/>
-    <xacro:property name="TrolleyPath" value="package://TestInput/urdf/model/1.STL"/>
-    <xacro:property name="Link1Path" value="package://TestInput/urdf/model/2.STL"/>
-    <xacro:property name="Link2Path" value="package://TestInput/urdf/model/3.STL"/>
-    <xacro:property name="Link3Path" value="package://TestInput/urdf/model/4.STL"/>
-    <xacro:property name="Link4Path" value="package://TestInput/urdf/model/5.STL"/>
-    <xacro:property name="Link5Path" value="package://TestInput/urdf/model/6.STL"/>
-    <xacro:property name="Link6Path" value="package://TestInput/urdf/model/7.STL"/>
+    <xacro:property name="TrolleyPath" value="package://model_source/urdf/model/1.STL"/>
+    <xacro:property name="Link1Path" value="package://model_source/urdf/model/2.STL"/>
+    <xacro:property name="Link2Path" value="package://model_source/urdf/model/3.STL"/>
+    <xacro:property name="Link3Path" value="package://model_source/urdf/model/4.STL"/>
+    <xacro:property name="Link4Path" value="package://model_source/urdf/model/5.STL"/>
+    <xacro:property name="Link5Path" value="package://model_source/urdf/model/6.STL"/>
+    <xacro:property name="Link6Path" value="package://model_source/urdf/model/7.STL"/>
     <link name="base_link">
         <visual>
             <geometry>
                 <mesh filename="${TrolleyPath}"/>
-                <!--                <box size="0.5 0.2 0.1" />-->
             </geometry>
             <origin rpy="0 0 0" xyz="0 0 0"/>
@@ -20,4 +19,10 @@
             </material>
         </visual>
+        <collision>
+            <origin xyx="0 0 0" rpy="0 0 0"/>
+            <geometry>
+                <mesh filename="${TrolleyPath}"/>
+            </geometry>
+        </collision>
     </link>
     <link name="link_1">
@@ -25,5 +30,4 @@
             <geometry>
                 <mesh filename="${Link1Path}"/>
-                <!--                <box size="0.5 0.2 0.1" />-->
             </geometry>
             <origin rpy="0 0 0" xyz="0 0 0"/>
@@ -32,4 +36,10 @@
             </material>
         </visual>
+        <collision>
+            <origin xyx="0 0 0" rpy="0 0 0"/>
+            <geometry>
+                <mesh filename="${Link1Path}"/>
+            </geometry>
+        </collision>
     </link>
     <joint name="BaseToLink_1" type="continuous">
@@ -38,4 +48,6 @@
         <origin xyz="0 0 0.375" rpy="${-PI/2} 0 0"/>
         <axis xyz="0 1 0"/>
+        <limit effort="300" velocity="1" lower="-2.96" upper="2.96"/>
+        <dynamics damping="50" friction="1"/>
     </joint>
     <link name="link_2">
@@ -49,4 +61,10 @@
             </material>
         </visual>
+        <collision>
+            <origin xyx="0 0 0" rpy="0 0 0"/>
+            <geometry>
+                <mesh filename="${Link2Path}"/>
+            </geometry>
+        </collision>
     </link>
     <joint name="Link_1ToLink_2" type="continuous">
@@ -55,4 +73,6 @@
         <origin xyz="0.0 0.0 0.0" rpy="0 0 0"/>
         <axis xyz="0 0 1"/>
+        <limit effort="300" velocity="1" lower="-2.96" upper="2.96"/>
+        <dynamics damping="50" friction="1"/>
     </joint>
     <link name="link_3">
@@ -66,4 +86,10 @@
             </material>
         </visual>
+        <collision>
+            <origin xyx="0 0 0" rpy="0 0 0"/>
+            <geometry>
+                <mesh filename="${Link3Path}"/>
+            </geometry>
+        </collision>
     </link>
     <joint name="Link_2ToLink_3" type="continuous">
@@ -72,4 +98,6 @@
         <origin xyz="0 -0.4 0.02" rpy="0 0 0"/>
         <axis xyz="0 0 1"/>
+        <limit effort="300" velocity="1" lower="-2.96" upper="2.96"/>
+        <dynamics damping="50" friction="1"/>
     </joint>
     <link name="link_4">
@@ -83,4 +111,10 @@
             </material>
         </visual>
+        <collision>
+            <origin xyx="0 0 0" rpy="0 0 0"/>
+            <geometry>
+                <mesh filename="${Link4Path}"/>
+            </geometry>
+        </collision>
     </link>
     <joint name="Link_3ToLink_4" type="continuous">
@@ -100,4 +134,10 @@
             </material>
         </visual>
+        <collision>
+            <origin xyx="0 0 0" rpy="0 0 0"/>
+            <geometry>
+                <mesh filename="${Link5Path}"/>
+            </geometry>
+        </collision>
     </link>
     <joint name="Link_4ToLink_5" type="continuous">
@@ -106,4 +146,6 @@
         <origin xyz="0 0 0.45" rpy="${-PI/2} 0 0"/>
         <axis xyz="0 0 1"/>
+        <limit effort="300" velocity="1" lower="-2.96" upper="2.96"/>
+        <dynamics damping="50" friction="1"/>
     </joint>
     <link name="link_6">
@@ -117,4 +159,10 @@
             </material>
         </visual>
+        <collision>
+            <origin xyx="0 0 0" rpy="0 0 0"/>
+            <geometry>
+                <mesh filename="${Link6Path}"/>
+            </geometry>
+        </collision>
     </link>
     <joint name="Link_5ToLink_6" type="continuous">
@@ -123,4 +171,6 @@
         <origin xyz="0 -0.07 0" rpy="${PI/2} 0 0"/>
         <axis xyz="0 0 1"/>
+        <limit effort="300" velocity="1" lower="-2.96" upper="2.96"/>
+        <dynamics damping="50" friction="1"/>
     </joint>
 </robot>
